Commit message: add robot wrapper

File: models/urdf/biped_robot_12dof.urdf (robot description, URDF)
Before this commit: robot biped 12-dof robot, 13 links, 12 joints
Joints:
- joint left_ankle_pitch_joint: limit lower=-0.5235987901687622 upper=0.5235987901687622 effort=1000.0 velocity=1000.0 -> lower=-0.5235987901687622 upper=0.5235987901687622 effort=30.0 velocity=60
- joint left_ankle_roll_joint: limit lower=-0.2617993950843811 upper=0.2617993950843811 effort=1000.0 velocity=1000.0 -> lower=-0.2617993950843811 upper=0.2617993950843811 effort=30.0 velocity=60
- joint left_hip_pitch_joint: limit lower=-1.0471975803375244 upper=1.0471975803375244 effort=1000.0 velocity=1000.0 -> lower=-1.0471975803375244 upper=1.0471975803375244 effort=48.0 velocity=60
- joint left_hip_roll_joint: limit lower=-0.7853981852531433 upper=1.0471975803375244 effort=1000.0 velocity=1000.0 -> lower=-0.7853981852531433 upper=1.0471975803375244 effort=48.0 velocity=60
- joint left_hip_yaw_joint: limit lower=-0.7853981852531433 upper=0.7853981852531433 effort=1000.0 velocity=1000.0 -> lower=-0.7853981852531433 upper=0.7853981852531433 effort=18.0 velocity=60
- joint left_knee_pitch_joint: limit lower=-0.1745329201221466 upper=2.094395160675049 effort=1000.0 velocity=1000.0 -> lower=-0.1745329201221466 upper=2.094395160675049 effort=48.0 velocity=60
- joint right_ankle_pitch_joint: limit lower=-0.5235987901687622 upper=0.5235987901687622 effort=1000.0 velocity=1000.0 -> lower=-0.5235987901687622 upper=0.5235987901687622 effort=30.0 velocity=60
- joint right_ankle_roll_joint: limit lower=-0.2617993950843811 upper=0.2617993950843811 effort=1000.0 velocity=1000.0 -> lower=-0.2617993950843811 upper=0.2617993950843811 effort=30.0 velocity=60
- joint right_hip_pitch_joint: limit lower=-1.0471975803375244 upper=1.0471975803375244 effort=1000.0 velocity=1000.0 -> lower=-1.0471975803375244 upper=1.0471975803375244 effort=48.0 velocity=60
- joint right_hip_roll_joint: limit lower=-1.0471975803375244 upper=0.6108652353286743 effort=1000.0 velocity=1000.0 -> lower=-1.0471975803375244 upper=0.6108652353286743 effort=48.0 velocity=60
- joint right_hip_yaw_joint: limit lower=-0.7853981852531433 upper=0.7853981852531433 effort=1000.0 velocity=1000.0 -> lower=-0.7853981852531433 upper=0.7853981852531433 effort=18.0 velocity=60
- joint right_knee_pitch_joint: limit lower=-0.1745329201221466 upper=2.094395160675049 effort=1000.0 velocity=1000.0 -> lower=-0.1745329201221466 upper=2.094395160675049 effort=48.0 velocity=60

File: models/urdf/left_leg_6dof.urdf (robot description, URDF)
Before this commit: robot biped 12-dof robot - left leg, 7 links, 6 joints
Joints:
- joint left_ankle_pitch_joint: limit lower=-0.5235987901687622 upper=0.5235987901687622 effort=1000.0 velocity=1000.0 -> lower=-0.5235987901687622 upper=0.5235987901687622 effort=1000.0 velocity=100
- joint left_ankle_roll_joint: limit lower=-0.2617993950843811 upper=0.2617993950843811 effort=1000.0 velocity=1000.0 -> lower=-0.2617993950843811 upper=0.2617993950843811 effort=1000.0 velocity=100
- joint left_hip_pitch_joint: limit lower=-1.0471975803375244 upper=1.0471975803375244 effort=1000.0 velocity=1000.0 -> lower=-1.0471975803375244 upper=1.0471975803375244 effort=48.0 velocity=100.0
- joint left_hip_roll_joint: limit lower=-0.7853981852531433 upper=1.0471975803375244 effort=1000.0 velocity=1000.0 -> lower=-0.7853981852531433 upper=1.0471975803375244 effort=48.0 velocity=100
- joint left_hip_yaw_joint: limit lower=-0.7853981852531433 upper=0.7853981852531433 effort=1000.0 velocity=1000.0 -> lower=-0.7853981852531433 upper=0.7853981852531433 effort=1000.0 velocity=100
- joint left_knee_pitch_joint: limit lower=-0.1745329201221466 upper=2.094395160675049 effort=1000.0 velocity=1000.0 -> lower=-0.1745329201221466 upper=2.094395160675049 effort=1000.0 velocity=100
